File: reform2-trackball-sensor-pcb/reform2-trackball-sensor.sch (KiCad schematic (older format))
At the start: 14 parts, among them J1 Conn_01x06_Male, U1 PAT9125EL

Commit message: Hardware changes for the mouse-trak
Parts:
- removed H1, H3, H4, H6: MountingHole, MountingHole:MountingHole_2.2mm_M2, symbol Mechanical:MountingHole
- J1: value Conn_01x06_Male -> Conn_01x05_Male; footprint Connector_FFC-FPC:Hirose_FH12-6S-0.5SH_1x06-1MP_P0.50mm_Horizontal -> Connector_PinHeader_2.54mm:PinHeader_1x05_P2.54mm_Horizontal; symbol Connector:Conn_01x06_Male -> Connector:Conn_01x05_Male
Connections:
- net +3V3: now also J1.5 (Pin_5); no longer J1.1 (Pin_1)
- net GND: now also J1.1 (Pin_1); no longer J1.6 (Pin_6)
- net MOTION: now also J1.2 (Pin_2); no longer J1.5 (Pin_5)
- net SCL: now also J1.4 (Pin_4); no longer J1.3 (Pin_3)
- net SDA: now also J1.3 (Pin_3); no longer J1.4 (Pin_4)
- no-connect marks 2 -> 1
Changed lines of the file:
@@
-$EndComp
-$Comp
-L Mechanical:MountingHole H1
-U 1 1 5D1F454C
-P 4100 4700
-F 0 "H1" H 4200 4746 50  0000 L CNN
-F 1 "MountingHole" H 4200 4655 50  0000 L CNN
-F 2 "MountingHole:MountingHole_2.2mm_M2" H 4100 4700 50  0001 C CNN
-F 3 "~" H 4100 4700 50  0001 C CNN
-F 4 "NOSTUFF" H 4100 4700 50  0001 C CNN "MFR"
-F 5 "NOSTUFF" H 4100 4700 50  0001 C CNN "MFR_NO"
-	1    4100 4700
-	1    0    0    -1
 $EndComp
 $Comp
@@
 $EndComp
 $Comp
-L Connector:Conn_01x06_Male J1
+L Connector:Conn_01x05_Male J1
 U 1 1 5D1E2C79
-P 7000 3700
-F 0 "J1" H 6972 3724 50  0000 R CNN
-F 1 "Conn_01x06_Male" H 6972 3633 50  0000 R CNN
-F 2 "Connector_FFC-FPC:Hirose_FH12-6S-0.5SH_1x06-1MP_P0.50mm_Horizontal" H 7000 3700 50  0001 C CNN
-F 3 "~" H 7000 3700 50  0001 C CNN
-F 4 "Hirose" H 7000 3700 50  0001 C CNN "MFR"
-F 5 "FH12-6S-0.5SH(55)" H 7000 3700 50  0001 C CNN "MFR_NO"
-	1    7000 3700
-	-1   0    0    1
+P 7000 3600
+F 0 "J1" H 6972 3624 50  0000 R CNN
+F 1 "Conn_01x05_Male" H 6972 3533 50  0000 R CNN
+F 2 "Connector_PinHeader_2.54mm:PinHeader_1x05_P2.54mm_Horizontal" H 7000 3600 50  0001 C CNN
+F 3 "~" H 7000 3600 50  0001 C CNN
+F 4 "Hirose" H 7000 3600 50  0001 C CNN "MFR"
+F 5 "FH12-6S-0.5SH(55)" H 7000 3600 50  0001 C CNN "MFR_NO"
+	1    7000 3600
+	-1   0    0    -1
 $EndComp
 $Comp
 L power:+3V3 #PWR0104
 U 1 1 5D1E8452
-P 6450 3900
-F 0 "#PWR0104" H 6450 3750 50  0001 C CNN
-F 1 "+3V3" V 6465 4028 50  0000 L CNN
-F 2 "" H 6450 3900 50  0001 C CNN
-F 3 "" H 6450 3900 50  0001 C CNN
-	1    6450 3900
+P 6450 3800
+F 0 "#PWR0104" H 6450 3650 50  0001 C CNN
+F 1 "+3V3" V 6465 3928 50  0000 L CNN
+F 2 "" H 6450 3800 50  0001 C CNN
+F 3 "" H 6450 3800 50  0001 C CNN
+	1    6450 3800
 	0    -1   -1   0
 $EndComp
-NoConn ~ 6800 3800
 Text Label 6500 3500 0    50   ~ 0
 MOTION
@@
 	6450 3400 6750 3400
 Wire Wire Line
-	6450 3900 6750 3900
+	6450 3800 6750 3800
 $Comp
 L power:PWR_FLAG #FLG0101
 U 1 1 5E567A57
-P 6750 3900
-F 0 "#FLG0101" H 6750 3975 50  0001 C CNN
-F 1 "PWR_FLAG" V 6750 4027 50  0000 L CNN
-F 2 "" H 6750 3900 50  0001 C CNN
-F 3 "~" H 6750 3900 50  0001 C CNN
-	1    6750 3900
+P 6750 3800
+F 0 "#FLG0101" H 6750 3875 50  0001 C CNN
+F 1 "PWR_FLAG" V 6750 3927 50  0000 L CNN
+F 2 "" H 6750 3800 50  0001 C CNN
+F 3 "~" H 6750 3800 50  0001 C CNN
+	1    6750 3800
 	-1   0    0    1
 $EndComp
-Connection ~ 6750 3900
+Connection ~ 6750 3800
 Wire Wire Line
-	6750 3900 6800 3900
+	6750 3800 6800 3800
 Wire Wire Line
 	3850 3200 3850 3400
@@
 	6750 3400 6800 3400
 $Comp
-L Mechanical:MountingHole H3
-U 1 1 5E56B94C
-P 4100 5350
-F 0 "H3" H 4200 5396 50  0000 L CNN
-F 1 "MountingHole" H 4200 5305 50  0000 L CNN
-F 2 "MountingHole:MountingHole_2.2mm_M2" H 4100 5350 50  0001 C CNN
-F 3 "~" H 4100 5350 50  0001 C CNN
-F 4 "NOSTUFF" H 4100 5350 50  0001 C CNN "MFR"
-F 5 "NOSTUFF" H 4100 5350 50  0001 C CNN "MFR_NO"
-	1    4100 5350
-	1    0    0    -1
-$EndComp
-$Comp
-L Mechanical:MountingHole H4
-U 1 1 5E56B958
-P 4100 5650
-F 0 "H4" H 4200 5696 50  0000 L CNN
-F 1 "MountingHole" H 4200 5605 50  0000 L CNN
-F 2 "MountingHole:MountingHole_2.2mm_M2" H 4100 5650 50  0001 C CNN
-F 3 "~" H 4100 5650 50  0001 C CNN
-F 4 "NOSTUFF" H 4100 5650 50  0001 C CNN "MFR"
-F 5 "NOSTUFF" H 4100 5650 50  0001 C CNN "MFR_NO"
-	1    4100 5650
-	1    0    0    -1
-$EndComp
-$Comp
 L Mechanical:MountingHole H5
 U 1 1 5E56C467
@@
 	1    0    0    -1
 $EndComp
-$Comp
-L Mechanical:MountingHole H6
-U 1 1 5E56C473
-P 5000 5000
-F 0 "H6" H 5100 5046 50  0000 L CNN
-F 1 "MountingHole" H 5100 4955 50  0000 L CNN
-F 2 "MountingHole:MountingHole_2.2mm_M2" H 5000 5000 50  0001 C CNN
-F 3 "~" H 5000 5000 50  0001 C CNN
-F 4 "NOSTUFF" H 5000 5000 50  0001 C CNN "MFR"
-F 5 "NOSTUFF" H 5000 5000 50  0001 C CNN "MFR_NO"
-	1    5000 5000
-	1    0    0    -1
-$EndComp
