File: reform2-trackball-pcb/reform2-trackball.sch (KiCad schematic (older format))
At the start: 42 parts, among them J1 Conn_USB, J2 Conn_01x06_Female, SW1 Choc, SW2 Choc, SW3 Choc, SW4 Choc, SW5 Choc, SW6 SW_RST, SW7 SW_HWB, U1 ATmega32U2-AU, U2 TLV75533PDBV, Y1 Crystal_GND24

Commit message: new pcb
Parts:
- removed MK10, MK11, MK12, MK5, MK6, MK9: Mounting_Hole, MountingHole:MountingHole_2.2mm_M2_Pad, symbol Mechanical:MountingHole_Pad
- removed MK13: LOGO, reform2-motherboard:mntreform, symbol Mechanical:MountingHole
- J2: value Conn_01x06_Female -> Conn_01x05_Female; footprint Connector_PinSocket_2.54mm:PinSocket_1x06_P2.54mm_Vertical -> Connector_PinSocket_2.54mm:PinSocket_1x05_P2.54mm_Vertical; symbol Connector:Conn_01x06_Female -> Connector:Conn_01x05_Female
- SW1: value Choc -> left; footprint keyswitches:PG1350 -> d_switchs:SubminiatureSPDT; symbol reform-trackball:Choc -> d_switchs:SubminiatureSPDT
- SW2: value Choc -> middle; footprint keyswitches:PG1350 -> d_switchs:SubminiatureSPDT; symbol reform-trackball:Choc -> d_switchs:SubminiatureSPDT
- SW3: value Choc -> right; footprint keyswitches:PG1350 -> d_switchs:SubminiatureSPDT; symbol reform-trackball:Choc -> d_switchs:SubminiatureSPDT
- SW4: value Choc -> btn4; footprint keyswitches:PG1350 -> Button_Switch_THT:Push_E-Switch_KS01Q01; symbol reform-trackball:Choc -> Switch:SW_Push
- SW5: value Choc -> btn5; footprint keyswitches:PG1350 -> Connector_PinHeader_2.54mm:PinHeader_1x02_P2.54mm_Vertical; symbol reform-trackball:Choc -> Switch:SW_Push
Connections:
- net GND: now also J2.5 (Pin_5), SW1.1 (COM), SW2.1 (COM), SW3.1 (COM), SW4.1, SW5.1; no longer J2.6 (Pin_6), SW1.2, SW2.2, SW3.2, SW4.2, SW5.2
- net MT: now also J2.4 (Pin_4); no longer J2.5 (Pin_5)
- net SCL: now also J2.2 (Pin_2); no longer J2.3 (Pin_3)
- net SDA: now also J2.3 (Pin_3); no longer J2.4 (Pin_4)
- net at U1.10 (PD4): now also SW1.3 (NO); no longer SW1.1
- net at U1.6 (PD0): now also SW5.2; no longer SW5.1
- net at U1.7 (PD1): now also SW4.2; no longer SW4.1
- net at U1.8 (PD2): now also SW3.3 (NO); no longer SW3.1
- net at U1.9 (PD3): now also SW2.3 (NO); no longer SW2.1
- no-connect marks 8 -> 10
Other:
- note added: "4th"
- note added: "ball"
- note added: "left"
- note added: "middle"
- note added: "right"
- moved on the sheet: SW4, SW5
